File: schematics/soundlabor_schloss.sch (KiCad schematic (older format))
At the start: 15 parts, among them P1 CONN_01X03, P2 CONN_01X02, P3 CONN_01X02, Q1 Q_NMOS_GDS, U1 4538

Commit message: Finishing basic PCB design. Feel free to improve on it. Uses a ground back plane and otherwise routes everything on front layer
Parts:
- 100k1: renamed from 100k2; footprint (none) -> Buttons_Switches_ThroughHole:SW_Micro_SPST
- 100k2: renamed from 100k1; footprint (none) -> Buttons_Switches_ThroughHole:SW_Micro_SPST
- 220µF1: renamed from 220µF2; footprint (none) -> Capacitors_Elko_ThroughHole:Elko_vert_11.2x6.3mm_RM2.5
- 220µF2: renamed from 220µF1; footprint (none) -> Capacitors_Elko_ThroughHole:Elko_vert_11.2x6.3mm_RM2.5
- D1: renamed from D2; footprint (none) -> LEDs:LED-5MM
- D2: renamed from D1; footprint (none) -> LEDs:LED-5MM
- D3: footprint (none) -> Diodes_ThroughHole:Diode_DO-35_SOD27_Horizontal_RM10
- P1: footprint (none) -> Pin_Headers:Pin_Header_Straight_1x03
- P2, P3: footprint (none) -> Pin_Headers:Pin_Header_Straight_1x02
- Q1: footprint (none) -> Housings_TO-92:TO-92_Molded_Wide
- R1: footprint (none) -> Resistors_SMD:R_1206_HandSoldering
Connections:
- net VSS is gone; now on net GND: 0.1µF1.1, P1.2 (P2), U1.8 (VSS), U1.8 (VSS)
- net GND: now also 10k1.2, 220µF2.2, U1.15 (gnd)
- net at P1.3 (P3), U1.12 (Clk+), U1.4 (Clk+): no longer 10k1.2
Other:
- moved on the sheet: 100k1, 10k1, P1

Commit message: pcb done
Parts:
- 0.1µF1: footprint Capacitors_SMD:C_1206_HandSoldering -> Capacitors_ThroughHole:C_Disc_D3_P2.5
- 100k1, 100k2: footprint Buttons_Switches_ThroughHole:SW_Micro_SPST -> Potentiometers:Potentiometer_Bourns_3006P_Angular_ScrewFront
- 10k1, R1: footprint Resistors_SMD:R_1206_HandSoldering -> Resistors_ThroughHole:Resistor_Horizontal_RM7mm
- 220µF1, 220µF2: footprint Capacitors_Elko_ThroughHole:Elko_vert_11.2x6.3mm_RM2.5 -> Capacitors_ThroughHole:C_Radial_D8_L11.5_P3.5
- D3: footprint Diodes_ThroughHole:Diode_DO-35_SOD27_Horizontal_RM10 -> Diodes_ThroughHole:Diode_DO-41_SOD81_Horizontal_RM10
- P1: footprint Pin_Headers:Pin_Header_Straight_1x03 -> Pin_Headers:Pin_Header_Angled_1x03
- P2: renamed from P3; footprint Pin_Headers:Pin_Header_Straight_1x02 -> Terminal_Blocks:TerminalBlock_Pheonix_MKDS1.5-2pol
- P3: renamed from P2; footprint Pin_Headers:Pin_Header_Straight_1x02 -> Terminal_Blocks:TerminalBlock_Pheonix_MKDS1.5-2pol
- Q1: footprint Housings_TO-92:TO-92_Molded_Wide -> TO_SOT_Packages_THT:TO-220_Neutral123_Vertical
- U1: footprint Housings_DIP:DIP-16_W7.62mm -> Housings_DIP:DIP-16_W7.62mm_LongPads
Connections:
- net GND: now also P3.2 (P2); no longer 10k1.2, P3.1 (P1)
- net at P1.3 (P3), U1.12 (Clk+), U1.4 (Clk+): now also 10k1.2
- net +12V: now reaches D3.1 (K), P2.1 (P1)
- net +12V: now also P3.1 (P1); no longer P3.2 (P2)
- no-connect marks 2 -> 3
Other:
- moved on the sheet: P3
Changed lines of the file:
@@
 F 0 "U1" H 2150 3250 60  0000 C CNN
 F 1 "4538" H 2300 2450 60  0000 C CNN
-F 2 "Housings_DIP:DIP-16_W7.62mm" H 2100 2850 60  0001 C CNN
+F 2 "Housings_DIP:DIP-16_W7.62mm_LongPads" H 2100 2850 60  0001 C CNN
 F 3 "" H 2100 2850 60  0000 C CNN
 	1    2100 2850
@@
 F 0 "220µF1" H 950 2500 50  0000 L CNN
 F 1 "CP" H 1275 2500 50  0000 L CNN
-F 2 "Capacitors_Elko_ThroughHole:Elko_vert_11.2x6.3mm_RM2.5" H 1288 2450 30  0001 C CNN
+F 2 "Capacitors_ThroughHole:C_Radial_D8_L11.5_P3.5" H 1288 2450 30  0001 C CNN
 F 3 "" H 1250 2600 60  0000 C CNN
 	1    1250 2600
@@
 F 0 "U1" H 4150 4050 60  0000 C CNN
 F 1 "4538" H 4300 3250 60  0000 C CNN
-F 2 "Housings_DIP:DIP-16_W7.62mm" H 4100 3650 60  0001 C CNN
+F 2 "Housings_DIP:DIP-16_W7.62mm_LongPads" H 4100 3650 60  0001 C CNN
 F 3 "" H 4100 3650 60  0000 C CNN
 	2    4100 3650
@@
 F 0 "0.1µF1" V 2250 3900 50  0000 L CNN
 F 1 "C" H 2325 3750 50  0000 L CNN
-F 2 "Capacitors_SMD:C_1206_HandSoldering" H 2338 3700 30  0001 C CNN
+F 2 "Capacitors_ThroughHole:C_Disc_D3_P2.5" H 2338 3700 30  0001 C CNN
 F 3 "" H 2300 3850 60  0000 C CNN
 	1    2300 3850
@@
 F 0 "220µF2" H 3050 3250 50  0000 L CNN
 F 1 "CP" H 3325 3250 50  0000 L CNN
-F 2 "Capacitors_Elko_ThroughHole:Elko_vert_11.2x6.3mm_RM2.5" H 3338 3200 30  0001 C CNN
+F 2 "Capacitors_ThroughHole:C_Radial_D8_L11.5_P3.5" H 3338 3200 30  0001 C CNN
 F 3 "" H 3300 3350 60  0000 C CNN
 	1    3300 3350
@@
 F 0 "100k2" H 3900 2750 50  0000 C CNN
 F 1 "POT" H 3900 2850 50  0000 C CNN
-F 2 "Buttons_Switches_ThroughHole:SW_Micro_SPST" H 3900 2850 60  0001 C CNN
+F 2 "Potentiometers:Potentiometer_Bourns_3006P_Angular_ScrewFront" H 3900 2850 60  0001 C CNN
 F 3 "" H 3900 2850 60  0000 C CNN
 	1    3900 2850
@@
 F 0 "100k1" H 1550 2150 50  0000 C CNN
 F 1 "POT" H 1550 2250 50  0000 C CNN
-F 2 "Buttons_Switches_ThroughHole:SW_Micro_SPST" H 1550 2250 60  0001 C CNN
+F 2 "Potentiometers:Potentiometer_Bourns_3006P_Angular_ScrewFront" H 1550 2250 60  0001 C CNN
 F 3 "" H 1550 2250 60  0000 C CNN
 	1    1550 2250
@@
 F 0 "10k1" V 2630 4550 50  0000 C CNN
 F 1 "R" V 2550 4550 50  0000 C CNN
-F 2 "Resistors_SMD:R_1206_HandSoldering" V 2480 4550 30  0001 C CNN
+F 2 "Resistors_ThroughHole:Resistor_Horizontal_RM7mm" V 2480 4550 30  0001 C CNN
 F 3 "" H 2550 4550 30  0000 C CNN
 	1    2550 4550
@@
 F 0 "P1" H 1400 4300 50  0000 C CNN
 F 1 "CONN_01X03" H 1550 3900 50  0000 C CNN
-F 2 "Pin_Headers:Pin_Header_Straight_1x03" H 1400 4100 60  0001 C CNN
+F 2 "Pin_Headers:Pin_Header_Angled_1x03" H 1400 4100 60  0001 C CNN
 F 3 "" H 1400 4100 60  0000 C CNN
 	1    1400 4100
@@
 L VCC #PWR02
 U 1 1 55F46611
-P 1750 4500
-F 0 "#PWR02" H 1750 4350 50  0001 C CNN
-F 1 "VCC" H 1750 4650 50  0000 C CNN
-F 2 "" H 1750 4500 60  0000 C CNN
-F 3 "" H 1750 4500 60  0000 C CNN
-	1    1750 4500
-	-1   0    0    1
+P 1550 4600
+F 0 "#PWR02" H 1550 4450 50  0001 C CNN
+F 1 "VCC" H 1550 4750 50  0000 C CNN
+F 2 "" H 1550 4600 60  0000 C CNN
+F 3 "" H 1550 4600 60  0000 C CNN
+	1    1550 4600
+	1    0    0    -1
 $EndComp
 $Comp
@@
 F 0 "Q1" H 5650 2950 50  0000 R CNN
 F 1 "Q_NMOS_GDS" H 6000 2850 50  0000 R CNN
-F 2 "Housings_TO-92:TO-92_Molded_Wide" H 5550 3000 29  0001 C CNN
+F 2 "TO_SOT_Packages_THT:TO-220_Neutral123_Vertical" H 5550 3000 29  0001 C CNN
 F 3 "" H 5350 2900 60  0000 C CNN
 	1    5350 2900
@@
 F 0 "R1" V 5280 3100 50  0000 C CNN
 F 1 "38k" V 5200 3100 50  0000 C CNN
-F 2 "Resistors_SMD:R_1206_HandSoldering" V 5130 3100 30  0001 C CNN
+F 2 "Resistors_ThroughHole:Resistor_Horizontal_RM7mm" V 5130 3100 30  0001 C CNN
 F 3 "" H 5200 3100 30  0000 C CNN
 	1    5200 3100
@@
 $EndComp
 $Comp
-L CONN_01X02 P3
+L CONN_01X02 P2
 U 1 1 55F4D3D8
 P 6400 2400
-F 0 "P3" H 6400 2550 50  0000 C CNN
+F 0 "P2" H 6400 2550 50  0000 C CNN
 F 1 "CONN_01X02" V 6500 2400 50  0000 C CNN
-F 2 "Pin_Headers:Pin_Header_Straight_1x02" H 6400 2400 60  0001 C CNN
+F 2 "Terminal_Blocks:TerminalBlock_Pheonix_MKDS1.5-2pol" H 6400 2400 60  0001 C CNN
 F 3 "" H 6400 2400 60  0000 C CNN
 	1    6400 2400
@@
 $EndComp
 $Comp
-L CONN_01X02 P2
+L CONN_01X02 P3
 U 1 1 55F4DA64
-P 6400 1800
-F 0 "P2" H 6400 1950 50  0000 C CNN
-F 1 "CONN_01X02" V 6500 1800 50  0000 C CNN
-F 2 "Pin_Headers:Pin_Header_Straight_1x02" H 6400 1800 60  0001 C CNN
-F 3 "" H 6400 1800 60  0000 C CNN
-	1    6400 1800
+P 6400 3000
+F 0 "P3" H 6400 3150 50  0000 C CNN
+F 1 "CONN_01X02" V 6500 3000 50  0000 C CNN
+F 2 "Terminal_Blocks:TerminalBlock_Pheonix_MKDS1.5-2pol" H 6400 3000 60  0001 C CNN
+F 3 "" H 6400 3000 60  0000 C CNN
+	1    6400 3000
 	1    0    0    -1
 $EndComp
@@
 F 0 "D3" H 6100 2300 50  0000 C CNN
 F 1 "D" H 6000 2250 50  0000 C CNN
-F 2 "Diodes_ThroughHole:Diode_DO-35_SOD27_Horizontal_RM10" H 6000 2350 60  0001 C CNN
+F 2 "Diodes_ThroughHole:Diode_DO-41_SOD81_Horizontal_RM10" H 6000 2350 60  0001 C CNN
 F 3 "" H 6000 2350 60  0000 C CNN
 	1    6000 2350
@@
 L VCC #PWR05
 U 1 1 55F52692
-P 3900 2600
-F 0 "#PWR05" H 3900 2450 50  0001 C CNN
-F 1 "VCC" H 3900 2750 50  0000 C CNN
-F 2 "" H 3900 2600 60  0000 C CNN
-F 3 "" H 3900 2600 60  0000 C CNN
-	1    3900 2600
+P 3900 2550
+F 0 "#PWR05" H 3900 2400 50  0001 C CNN
+F 1 "VCC" H 3900 2700 50  0000 C CNN
+F 2 "" H 3900 2550 60  0000 C CNN
+F 3 "" H 3900 2550 60  0000 C CNN
+	1    3900 2550
 	1    0    0    -1
 $EndComp
@@
 L GND #PWR07
 U 1 1 55F5312C
-P 3550 2550
-F 0 "#PWR07" H 3550 2300 50  0001 C CNN
-F 1 "GND" H 3550 2400 50  0000 C CNN
-F 2 "" H 3550 2550 60  0000 C CNN
-F 3 "" H 3550 2550 60  0000 C CNN
-	1    3550 2550
-	0    -1   -1   0
+P 3550 2650
+F 0 "#PWR07" H 3550 2400 50  0001 C CNN
+F 1 "GND" H 3550 2500 50  0000 C CNN
+F 2 "" H 3550 2650 60  0000 C CNN
+F 3 "" H 3550 2650 60  0000 C CNN
+	1    3550 2650
+	1    0    0    -1
 $EndComp
 NoConn ~ 4150 2850
 NoConn ~ 1800 2250
+Text Label 6150 2950 2    60   ~ 0
++12V
+Text Label 6150 3050 2    60   ~ 0
+GND
+Text Label 6650 2300 0    60   ~ 0
+LOCK+
+Text Label 6650 2450 0    60   ~ 0
+LOCK-
+Text Label 1150 4100 2    60   ~ 0
+GND
+Text Label 1150 4200 2    60   ~ 0
+VCC
+Text Label 1150 4000 2    60   ~ 0
+PI
 Wire Wire Line
 	1300 3750 3500 3750
@@
 Wire Wire Line
 	2100 4200 2100 3500
-Wire Wire Line
-	1900 3200 1900 4100
 Connection ~ 1900 4100
 Wire Wire Line
@@
 Connection ~ 3300 3100
 Wire Wire Line
-	3300 3500 3300 4100
+	3300 3500 3300 4500
 Wire Wire Line
 	4700 3350 5000 3350
@@
 	5450 3100 5450 3500
 Wire Wire Line
-	5400 3350 6050 3350
+	5400 3350 6150 3350
 Connection ~ 5450 3350
 Wire Wire Line
@@
 Wire Wire Line
 	6200 2350 6150 2350
-Wire Wire Line
-	6150 1850 6200 1850
-Wire Wire Line
-	6200 1750 6050 1750
-Wire Wire Line
-	6050 1750 6050 3350
 Connection ~ 5800 2450
 Wire Wire Line
@@
 	5800 2350 5850 2350
 Wire Wire Line
-	6150 2350 6150 1850
-Connection ~ 6150 2350
-Wire Wire Line
 	1750 3850 2150 3850
 Wire Wire Line
-	2450 3850 2550 3850
-Wire Wire Line
-	2550 3850 2550 4400
-Connection ~ 2550 4100
-Wire Wire Line
-	3900 2600 3900 2700
+	2450 3850 2750 3850
+Wire Wire Line
+	3900 2550 3900 2700
 Wire Wire Line
 	1550 1950 1550 2100
@@
 	3550 2550 3400 2550
 Wire Wire Line
-	1750 3850 1750 4500
+	1750 3850 1750 4750
 Connection ~ 1750 4200
 Wire Wire Line
@@
 Connection ~ 2850 4350
 Wire Wire Line
-	2550 4850 2550 4700
+	2550 4700 2550 4850
 Wire Wire Line
 	2850 3000 2850 4350
@@
 Connection ~ 3300 4100
 Connection ~ 3300 3550
+Connection ~ 6150 2350
+Wire Wire Line
+	6150 2350 6150 2950
+Wire Wire Line
+	6150 2950 6200 2950
+Wire Wire Line
+	6200 3050 6150 3050
+Wire Wire Line
+	6150 3050 6150 3350
+Connection ~ 2550 4000
+Wire Wire Line
+	3550 2550 3550 2650
+Wire Wire Line
+	1750 4750 1550 4750
+Wire Wire Line
+	1550 4750 1550 4600
+NoConn ~ 4700 3950
+$Comp
+L GND #PWR08
+U 1 1 56FF3495
+P 3300 4500
+F 0 "#PWR08" H 3300 4250 50  0001 C CNN
+F 1 "GND" H 3300 4350 50  0000 C CNN
+F 2 "" H 3300 4500 50  0000 C CNN
+F 3 "" H 3300 4500 50  0000 C CNN
+	1    3300 4500
+	1    0    0    -1
+$EndComp
+Wire Wire Line
+	1900 4100 1900 3200
+Wire Wire Line
+	2550 4400 2550 4000
+Wire Wire Line
+	2750 3850 2750 4100
+Connection ~ 2750 4100
 $EndSCHEMATC

Commit message: improved circuit
Parts:
- added C1: 3300µ, symbol CP
- added R1, R3: 120R, symbol R
- R2: renamed from R1; value 38k -> 100k
- renumbered P3 to P2, P2 to P3
Connections:
- net +12V: now also C1.1
- net GND: now also C1.2; no longer D2.1 (K)
- net VCC: now also R3.1
- net at U1.6 (Q): now also R1.2; no longer D1.2 (A)
- net at Q1.1 (G), R2.2, U1.10 (Q): no longer D2.2 (A)
- net at D3.2 (A), P3.2 (P2), Q1.2 (D): now also D2.1 (K)
- new net: D2.2 (A), R3.2
- new net: D1.2 (A), R1.1
Other:
- moved on the sheet: D1, D2, D3, P2, P3, Q1, R2

Commit message: final version
Parts:
- C1: footprint (none) -> raspberrylock_lib:ECA1EM332
- R1, R3: footprint (none) -> Resistors_ThroughHole:Resistor_Horizontal_RM7mm
Connections:
- net PI: now also 10k1.2, P1.3 (P3), U1.12 (Clk+), U1.4 (Clk+)
- net at 220µF2.1, U1.14 (RxCx): now also 100k2.3; no longer 100k2.1
Other:
- moved on the sheet: 0.1µF1, 100k1, 100k2, 10k1, 220µF1, D1, P1, R1
